File: Ovve_Leds/R_letter.kicad_sch (KiCad schematic)
At the start: 0 parts

Commit message: Finished preliminary schematics
Parts:
- added D13, D14, D15, D16, D17, D18, D19, D20, D21, D22: LED, symbol Device:LED
- added H13, H14, H15, H16, H17, H18: MountingHole, symbol Mechanical:MountingHole
- added R13, R14, R15, R16, R17, R18, R19, R20, R21, R22: 150, symbol Device:R
- added U2: 74LS174, symbol 74xx:74LS174
Connections:
- net CLK_in_R: now also U2.9 (Cp)
- net DATA_in_R: now also U2.3 (D0)
- net DATA_out_R: now also R21.1, R22.1, U2.12 (Q4)
- new net: D16.2 (A), R16.2
- new net: D14.2 (A), R14.2
- new net: D22.2 (A), R22.2
- new net: D17.2 (A), R17.2
- new net: D21.2 (A), R21.2
- new net: D13.2 (A), R13.2
- new net: D15.2 (A), R15.2
- new net: D20.2 (A), R20.2
- new net: D19.2 (A), R19.2
- new net: D18.2 (A), R18.2
- new net +5V: U2.1 (~{Mr}), U2.16 (VCC)
- new net GND: D13.1 (K), D14.1 (K), D15.1 (K), D16.1 (K), D17.1 (K), D18.1 (K), D19.1 (K), D20.1 (K), D21.1 (K), D22.1 (K), U2.8 (GND)
- new net LED1: R13.1, R14.1, U2.2 (Q0), U2.4 (D1)
- new net LED2: R15.1, R16.1, U2.5 (Q1), U2.6 (D2)
- new net LED3: R17.1, R18.1, U2.11 (D3), U2.7 (Q2)
- new net LED4: R19.1, R20.1, U2.10 (Q3), U2.13 (D4)
- no-connect marks 0 -> 2

Commit message: Added decoupling capacitors and assigned footprints
Parts:
- added C3: 0.1u, Capacitor_SMD:C_0603_1608Metric, symbol Device:C
- D13, D14, D15, D16, D17, D18, D19, D20, D21, D22: footprint (none) -> LED_THT:LED_D5.0mm
- H13, H14, H15, H16, H17, H18: footprint (none) -> MountingHole:MountingHole_5.3mm_M5_DIN965_Pad
- R13, R14, R15, R16, R17, R18, R19, R20, R21, R22: footprint (none) -> Resistor_SMD:R_0603_1608Metric
- U2: footprint (none) -> Package_DIP:DIP-16_W7.62mm
Connections:
- net +5V: now also C3.1
- net GND: now also C3.2

Commit message: Updated flip-flops
Connections:
- net GND: now also U2.14 (D5)
- no-connect marks 2 -> 1
Changed lines of the file:
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@@
 		(at 86.36 73.66)
 	)
-	(no_connect
-		(at 41.91 73.66)
-	)
 	(wire
 		(pts
@@
 					(unit 1)
 				)
+			)
+		)
+	)
+	(symbol
+		(lib_id "power:GND")
+		(at 41.91 73.66 0)
+		(unit 1)
+		(exclude_from_sim no)
+		(in_bom yes)
+		(on_board yes)
+		(dnp no)
+		(property "Reference" "#PWR073"
+			(at 41.91 80.01 0)
+			(effects
+				(font
+					(size 1.27 1.27)
+				)
+				(hide yes)
+			)
+		)
+		(property "Value" "GND"
+			(at 41.91 77.47 0)
+			(effects
+				(font
+					(size 1.27 1.27)
+				)
+			)
+		)
+		(property "Footprint" ""
+			(at 41.91 73.66 0)
+			(effects
+				(font
+					(size 1.27 1.27)
+				)
+				(hide yes)
+			)
+		)
+		(property "Datasheet" ""
+			(at 41.91 73.66 0)
+			(effects
+				(font
+					(size 1.27 1.27)
+				)
+				(hide yes)
+			)
+		)
+		(property "Description" "Power symbol creates a global label with name \"GND\" , ground"
+			(at 41.91 73.66 0)
+			(effects
+				(font
+					(size 1.27 1.27)
+				)
+				(hide yes)
+			)
+		)
+		(pin "1"
+		)
+		(instances
+			(project "Ovve_Leds"
+				(path "/a3f154e4-ded7-4c3a-b779-1e1dc74aad12/304f816e-a663-4998-b1af-381b08366ecd"
+					(reference "#PWR073")
+					(unit 1)
+				)

Commit message: Component layout on PCB
Parts:
- removed H15, H16: MountingHole, MountingHole:MountingHole_5.3mm_M5_DIN965_Pad, symbol Mechanical:MountingHole
- renumbered H13 to H15, H14 to H16, H17 to H19, H18 to H20
Changed lines of the file:
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@@
 		(dnp no)
 		(fields_autoplaced yes)
-		(property "Reference" "H14"
+		(property "Reference" "H16"
 			(at 194.31 26.6699 0)
 			(effects
@@
 			(project "Ovve_Leds"
 				(path "/a3f154e4-ded7-4c3a-b779-1e1dc74aad12/304f816e-a663-4998-b1af-381b08366ecd"
-					(reference "H14")
+					(reference "H16")
 					(unit 1)
 				)
@@
 		(dnp no)
 		(fields_autoplaced yes)
-		(property "Reference" "H18"
+		(property "Reference" "H20"
 			(at 194.31 49.5299 0)
 			(effects
@@
 			(project "Ovve_Leds"
 				(path "/a3f154e4-ded7-4c3a-b779-1e1dc74aad12/304f816e-a663-4998-b1af-381b08366ecd"
-					(reference "H18")
+					(reference "H20")
 					(unit 1)
 				)
@@
 		(dnp no)
 		(fields_autoplaced yes)
-		(property "Reference" "H17"
+		(property "Reference" "H19"
 			(at 194.31 44.4499 0)
 			(effects
@@
 			(project "Ovve_Leds"
 				(path "/a3f154e4-ded7-4c3a-b779-1e1dc74aad12/304f816e-a663-4998-b1af-381b08366ecd"
-					(reference "H17")
+					(reference "H19")
 					(unit 1)
 				)
@@
 		(dnp no)
 		(fields_autoplaced yes)
-		(property "Reference" "H13"
+		(property "Reference" "H15"
 			(at 194.31 21.5899 0)
 			(effects
@@
 			(project "Ovve_Leds"
 				(path "/a3f154e4-ded7-4c3a-b779-1e1dc74aad12/304f816e-a663-4998-b1af-381b08366ecd"
-					(reference "H13")
+					(reference "H15")
 					(unit 1)
 				)
@@
 	)
 	(symbol
-		(lib_id "Mechanical:MountingHole")
-		(at 191.77 34.29 0)
-		(unit 1)
-		(exclude_from_sim yes)
-		(in_bom no)
-		(on_board yes)
-		(dnp no)
-		(fields_autoplaced yes)
-		(property "Reference" "H15"
-			(at 194.31 33.0199 0)
-			(effects
-				(font
-					(size 1.27 1.27)
-				)
-				(justify left)
-			)
-		)
-		(property "Value" "MountingHole"
-			(at 194.31 35.5599 0)
-			(effects
-				(font
-					(size 1.27 1.27)
-				)
-				(justify left)
-			)
-		)
-		(property "Footprint" "MountingHole:MountingHole_5.3mm_M5_DIN965_Pad"
-			(at 191.77 34.29 0)
-			(effects
-				(font
-					(size 1.27 1.27)
-				)
-				(hide yes)
-			)
-		)
-		(property "Datasheet" "~"
-			(at 191.77 34.29 0)
-			(effects
-				(font
-					(size 1.27 1.27)
-				)
-				(hide yes)
-			)
-		)
-		(property "Description" "Mounting Hole without connection"
-			(at 191.77 34.29 0)
-			(effects
-				(font
-					(size 1.27 1.27)
-				)
-				(hide yes)
-			)
-		)
-		(instances
-			(project "Ovve_Leds"
-				(path "/a3f154e4-ded7-4c3a-b779-1e1dc74aad12/304f816e-a663-4998-b1af-381b08366ecd"
-					(reference "H15")
-					(unit 1)
-				)
-			)
-		)
-	)
-	(symbol
 		(lib_id "Device:R")
 		(at 142.24 88.9 0)
@@
 					(unit 1)
 				)
-			)
-		)
-	)
-	(symbol
-		(lib_id "Mechanical:MountingHole")
-		(at 191.77 39.37 0)
-		(unit 1)
-		(exclude_from_sim yes)
-		(in_bom no)
-		(on_board yes)
-		(dnp no)
-		(fields_autoplaced yes)
-		(property "Reference" "H16"
-			(at 194.31 38.0999 0)
-			(effects
-				(font
-					(size 1.27 1.27)
-				)
-				(justify left)
-			)
-		)
-		(property "Value" "MountingHole"
-			(at 194.31 40.6399 0)
-			(effects
-				(font
-					(size 1.27 1.27)
-				)
-				(justify left)
-			)
-		)
-		(property "Footprint" "MountingHole:MountingHole_5.3mm_M5_DIN965_Pad"
-			(at 191.77 39.37 0)
-			(effects
-				(font
-					(size 1.27 1.27)
-				)
-				(hide yes)
-			)
-		)
-		(property "Datasheet" "~"
-			(at 191.77 39.37 0)
-			(effects
-				(font
-					(size 1.27 1.27)
-				)
-				(hide yes)
-			)
-		)
-		(property "Description" "Mounting Hole without connection"
-			(at 191.77 39.37 0)
-			(effects
-				(font
-					(size 1.27 1.27)
-				)
-				(hide yes)
-			)
-		)
-		(instances
-			(project "Ovve_Leds"
-				(path "/a3f154e4-ded7-4c3a-b779-1e1dc74aad12/304f816e-a663-4998-b1af-381b08366ecd"
-					(reference "H16")
-					(unit 1)
-				)
