File: Ovve_Leds/Arduino_Power_A_letter.kicad_sch (KiCad schematic)
At the start: 2 parts, among them J1 Conn_01x04

Commit message: Finished preliminary schematics
Parts:
- added D30, D31, D32, D33, D34, D35, D36, D37, D38: LED, symbol Device:LED
- added D39: D, symbol Device:D
- added H1, H2, H3, H4, H5, H6: MountingHole, symbol Mechanical:MountingHole
- added R30, R31, R32, R33, R34, R35, R36, R37, R38: 150, symbol Device:R
- added U4: 74LS174, symbol 74xx:74LS174
Connections:
- net CLK_out_K: now also A1.6 (D3), U4.9 (Cp)
- net DATA_out_K: now also R37.1, R38.1, U4.12 (Q4)
- net +5V: now reaches A1.27 (+5V)
- net +5V: now also D39.1 (K), U4.1 (~{Mr}), U4.16 (VCC)
- net GND: now reaches A1.29 (GND)
- net GND: now also A1.4 (GND), D30.1 (K), D31.1 (K), D32.1 (K), D33.1 (K), D34.1 (K), D35.1 (K), D36.1 (K), D37.1 (K), D38.1 (K), U4.8 (GND)
- net DATA: now reaches A1.5 (D2)
- net DATA: now also U4.3 (D0)
- new net: D35.2 (A), R35.2
- new net: D38.2 (A), R38.2
- new net: D33.2 (A), R33.2
- new net: D36.2 (A), R36.2
- new net: D30.2 (A), R30.2
- new net: D37.2 (A), R37.2
- new net: D31.2 (A), R31.2
- new net: D34.2 (A), R34.2
- new net: D32.2 (A), R32.2
- new net 6V_in: D39.2 (A)
- new net LED1: R30.1, R31.1, U4.2 (Q0), U4.4 (D1)
- new net LED2: R32.1, R33.1, U4.5 (Q1), U4.6 (D2)
- new net LED3: R34.1, U4.11 (D3), U4.7 (Q2)
- new net LED4: R35.1, R36.1, U4.10 (Q3), U4.13 (D4)
- no-connect marks 0 -> 27
Other:
- moved on the sheet: A1

Commit message: Added decoupling capacitors and assigned footprints
Parts:
- added C1: 0.1u, Capacitor_SMD:C_0603_1608Metric, symbol Device:C
- D30, D31, D32, D33, D34, D35, D36, D37, D38: footprint (none) -> LED_THT:LED_D5.0mm
- D39: footprint (none) -> Diode_THT:D_DO-201AD_P15.24mm_Horizontal
- H1, H2, H3, H4, H5, H6: footprint (none) -> MountingHole:MountingHole_5.3mm_M5_DIN965_Pad
- J1: footprint (none) -> Connector_PinHeader_2.54mm:PinHeader_1x04_P2.54mm_Horizontal
- R30, R31, R32, R33, R34, R35, R36, R37, R38: footprint (none) -> Resistor_SMD:R_0603_1608Metric
- U4: footprint (none) -> Package_DIP:DIP-16_W7.62mm
Connections:
- net +5V: now also C1.1
- net GND: now also C1.2
Changed lines of the file:
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@@
 	)
 	(junction
+		(at 190.5 57.15)
+		(diameter 0)
+		(color 0 0 0 0)
+	)
+	(junction
 		(at 43.18 124.46)
 		(diameter 0)
@@
 	(wire
 		(pts
+			(xy 196.85 57.15) (xy 190.5 57.15)
+		)
+		(stroke
+			(width 0)
+			(type default)
+		)
+	)
+	(wire
+		(pts
 			(xy 242.57 74.93) (xy 242.57 77.47)
 		)
@@
 	(wire
 		(pts
+			(xy 190.5 54.61) (xy 190.5 57.15)
+		)
+		(stroke
+			(width 0)
+			(type default)
+		)
+	)
+	(wire
+		(pts
+			(xy 190.5 57.15) (xy 190.5 62.23)
+		)
+		(stroke
+			(width 0)
+			(type default)
+		)
+	)
+	(wire
+		(pts
 			(xy 242.57 19.05) (xy 267.97 19.05)
 		)
@@
 			)
 		)
-		(property "Footprint" ""
+		(property "Footprint" "Resistor_SMD:R_0603_1608Metric"
 			(at 240.792 109.22 90)
 			(effects
@@
 			)
 		)
-		(property "Footprint" ""
+		(property "Footprint" "LED_THT:LED_D5.0mm"
 			(at 267.97 148.59 0)
 			(effects
@@
 			)
 		)
-		(property "Footprint" ""
+		(property "Footprint" "LED_THT:LED_D5.0mm"
 			(at 255.27 60.96 0)
 			(effects
@@
 			)
 		)
-		(property "Footprint" ""
+		(property "Footprint" "MountingHole:MountingHole_5.3mm_M5_DIN965_Pad"
 			(at 102.87 54.61 0)
 			(effects
@@
 			)
 		)
-		(property "Footprint" ""
+		(property "Footprint" "Resistor_SMD:R_0603_1608Metric"
 			(at 253.492 53.34 90)
 			(effects
@@
 			)
 		)
-		(property "Footprint" ""
+		(property "Footprint" "Resistor_SMD:R_0603_1608Metric"
 			(at 253.492 109.22 90)
 			(effects
@@
 			)
 		)
-		(property "Footprint" ""
+		(property "Footprint" "MountingHole:MountingHole_5.3mm_M5_DIN965_Pad"
 			(at 102.87 26.67 0)
 			(effects
@@
 			)
 		)
-		(property "Footprint" ""
+		(property "Footprint" "Resistor_SMD:R_0603_1608Metric"
 			(at 266.192 140.97 90)
 			(effects
@@
 			)
 		)
-		(property "Footprint" ""
+		(property "Footprint" "MountingHole:MountingHole_5.3mm_M5_DIN965_Pad"
 			(at 102.87 38.1 0)
 			(effects
@@
 			)
 		)
-		(property "Footprint" ""
+		(property "Footprint" "Resistor_SMD:R_0603_1608Metric"
 			(at 240.792 25.4 90)
 			(effects
@@
 			)
 		)
-		(property "Footprint" ""
+		(property "Footprint" "MountingHole:MountingHole_5.3mm_M5_DIN965_Pad"
 			(at 102.87 31.75 0)
 			(effects
@@
 			)
 		)
-		(property "Footprint" ""
+		(property "Footprint" "Connector_PinHeader_2.54mm:PinHeader_1x04_P2.54mm_Horizontal"
 			(at 267.97 135.89 0)
 			(effects
@@
 	(symbol
 		(lib_id "power:+5V")
-		(at 190.5 62.23 0)
+		(at 190.5 54.61 0)
 		(unit 1)
 		(exclude_from_sim no)
@@
 		(dnp no)
 		(property "Reference" "#PWR050"
-			(at 190.5 66.04 0)
+			(at 190.5 58.42 0)
 			(effects
 				(font
@@
 		)
 		(property "Value" "+5V"
-			(at 190.5 58.42 0)
+			(at 190.5 50.8 0)
 			(effects
 				(font
@@
 		)
 		(property "Footprint" ""
-			(at 190.5 62.23 0)
+			(at 190.5 54.61 0)
 			(effects
 				(font
@@
 		)
 		(property "Datasheet" ""
-			(at 190.5 62.23 0)
+			(at 190.5 54.61 0)
 			(effects
 				(font
@@
 		)
 		(property "Description" "Power symbol creates a global label with name \"+5V\""
-			(at 190.5 62.23 0)
+			(at 190.5 54.61 0)
 			(effects
 				(font
@@
 			)
 		)
-		(property "Footprint" ""
+		(property "Footprint" "Diode_THT:D_DO-201AD_P15.24mm_Horizontal"
 			(at 66.04 124.46 0)
 			(effects
@@
 			)
 		)
-		(property "Footprint" ""
+		(property "Footprint" "LED_THT:LED_D5.0mm"
 			(at 242.57 148.59 0)
 			(effects
@@
 			)
 		)
-		(property "Footprint" ""
+		(property "Footprint" "LED_THT:LED_D5.0mm"
 			(at 267.97 33.02 0)
 			(effects
@@
 			)
 		)
-		(property "Footprint" ""
+		(property "Footprint" "Resistor_SMD:R_0603_1608Metric"
 			(at 240.792 140.97 90)
 			(effects
@@
 			)
 		)
-		(property "Footprint" ""
+		(property "Footprint" "LED_THT:LED_D5.0mm"
 			(at 242.57 88.9 0)
 			(effects
@@
 			)
 		)
-		(property "Footprint" ""
+		(property "Footprint" "Resistor_SMD:R_0603_1608Metric"
 			(at 266.192 25.4 90)
 			(effects
@@
 			)
 		)
-		(property "Footprint" ""
+		(property "Footprint" "MountingHole:MountingHole_5.3mm_M5_DIN965_Pad"
 			(at 102.87 49.53 0)
 			(effects
@@
 			)
 		)
-		(property "Footprint" ""
+		(property "Footprint" "MountingHole:MountingHole_5.3mm_M5_DIN965_Pad"
 			(at 102.87 43.18 0)
 			(effects
@@
 	)
 	(symbol
+		(lib_id "power:GND")
+		(at 204.47 57.15 90)
+		(unit 1)
+		(exclude_from_sim no)
+		(in_bom yes)
+		(on_board yes)
+		(dnp no)
+		(fields_autoplaced yes)
+		(property "Reference" "#PWR067"
+			(at 210.82 57.15 0)
+			(effects
+				(font
+					(size 1.27 1.27)
+				)
+				(hide yes)
+			)
+		)
+		(property "Value" "GND"
+			(at 208.28 57.1499 90)
+			(effects
+				(font
+					(size 1.27 1.27)
+				)
+				(justify right)
+			)
+		)
+		(property "Footprint" ""
+			(at 204.47 57.15 0)
+			(effects
+				(font
+					(size 1.27 1.27)
+				)
+				(hide yes)
+			)
+		)
+		(property "Datasheet" ""
+			(at 204.47 57.15 0)
+			(effects
+				(font
+					(size 1.27 1.27)
+				)
+				(hide yes)
+			)
+		)
+		(property "Description" "Power symbol creates a global label with name \"GND\" , ground"
+			(at 204.47 57.15 0)
+			(effects
+				(font
+					(size 1.27 1.27)
+				)
+				(hide yes)
+			)
+		)
+		(pin "1"
+		)
+		(instances
+			(project "Ovve_Leds"
+				(path "/a3f154e4-ded7-4c3a-b779-1e1dc74aad12/7922422b-804d-4651-8572-e2719e6393b3"
+					(reference "#PWR067")
+					(unit 1)
+				)
+			)
+		)
+	)
+	(symbol
+		(lib_id "Device:C")
+		(at 200.66 57.15 90)
+		(unit 1)
+		(exclude_from_sim no)
+		(in_bom yes)
+		(on_board yes)
+		(dnp no)
+		(fields_autoplaced yes)
+		(property "Reference" "C1"
+			(at 200.66 49.53 90)
+			(effects
+				(font
+					(size 1.27 1.27)
+				)
+			)
+		)
+		(property "Value" "0.1u"
+			(at 200.66 52.07 90)
+			(effects
+				(font
+					(size 1.27 1.27)
+				)
+			)
+		)
+		(property "Footprint" "Capacitor_SMD:C_0603_1608Metric"
+			(at 204.47 56.1848 0)
+			(effects
+				(font
+					(size 1.27 1.27)
+				)
+				(hide yes)
+			)
+		)
+		(property "Datasheet" "~"
+			(at 200.66 57.15 0)
+			(effects
+				(font
+					(size 1.27 1.27)
+				)
+				(hide yes)
+			)
+		)
+		(property "Description" "Unpolarized capacitor"
+			(at 200.66 57.15 0)
+			(effects
+				(font
+					(size 1.27 1.27)
+				)
+				(hide yes)
+			)
+		)
+		(pin "1"
+		)
+		(pin "2"
+		)
+		(instances
+			(project "Ovve_Leds"
+				(path "/a3f154e4-ded7-4c3a-b779-1e1dc74aad12/7922422b-804d-4651-8572-e2719e6393b3"
+					(reference "C1")
+					(unit 1)
+				)
+			)
+		)
+	)
+	(symbol
 		(lib_id "Device:LED")
 		(at 242.57 60.96 90)
@@
 			)
 		)
-		(property "Footprint" ""
+		(property "Footprint" "LED_THT:LED_D5.0mm"
 			(at 242.57 60.96 0)
 			(effects
@@
 			)
 		)
-		(property "Footprint" ""
+		(property "Footprint" "LED_THT:LED_D5.0mm"
 			(at 242.57 33.02 0)
 			(effects
@@
 			)
 		)
-		(property "Footprint" ""
+		(property "Footprint" "Resistor_SMD:R_0603_1608Metric"
 			(at 240.792 81.28 90)
 			(effects
@@
 			)
 		)
-		(property "Footprint" ""
+		(property "Footprint" "LED_THT:LED_D5.0mm"
 			(at 255.27 116.84 0)
 			(effects
@@
 			)
 		)
-		(property "Footprint" ""
+		(property "Footprint" "Resistor_SMD:R_0603_1608Metric"
 			(at 240.792 53.34 90)
 			(effects
@@
 			)
 		)
-		(property "Footprint" ""
+		(property "Footprint" "LED_THT:LED_D5.0mm"
 			(at 242.57 116.84 0)
 			(effects
@@
 			)
 		)
-		(property "Footprint" ""
+		(property "Footprint" "Package_DIP:DIP-16_W7.62mm"
 			(at 190.5 80.01 0)
 			(effects

Commit message: Updated flip-flops
Connections:
- net GND: now also U4.14 (D5)
- no-connect marks 27 -> 26
Changed lines of the file:
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@@
 	)
 	(no_connect
-		(at 170.18 82.55)
-	)
-	(no_connect
 		(at 69.85 54.61)
 	)
@@
 					(unit 1)
 				)
+			)
+		)
+	)
+	(symbol
+		(lib_id "power:GND")
+		(at 170.18 82.55 0)
+		(unit 1)
+		(exclude_from_sim no)
+		(in_bom yes)
+		(on_board yes)
+		(dnp no)
+		(property "Reference" "#PWR072"
+			(at 170.18 88.9 0)
+			(effects
+				(font
+					(size 1.27 1.27)
+				)
+				(hide yes)
+			)
+		)
+		(property "Value" "GND"
+			(at 170.18 86.36 0)
+			(effects
+				(font
+					(size 1.27 1.27)
+				)
+			)
+		)
+		(property "Footprint" ""
+			(at 170.18 82.55 0)
+			(effects
+				(font
+					(size 1.27 1.27)
+				)
+				(hide yes)
+			)
+		)
+		(property "Datasheet" ""
+			(at 170.18 82.55 0)
+			(effects
+				(font
+					(size 1.27 1.27)
+				)
+				(hide yes)
+			)
+		)
+		(property "Description" "Power symbol creates a global label with name \"GND\" , ground"
+			(at 170.18 82.55 0)
+			(effects
+				(font
+					(size 1.27 1.27)
+				)
+				(hide yes)
+			)
+		)
+		(pin "1"
+		)
+		(instances
+			(project "Ovve_Leds"
+				(path "/a3f154e4-ded7-4c3a-b779-1e1dc74aad12/7922422b-804d-4651-8572-e2719e6393b3"
+					(reference "#PWR072")
+					(unit 1)
+				)

Commit message: Component layout on PCB
Parts:
- removed H4, H5, H6: MountingHole, MountingHole:MountingHole_5.3mm_M5_DIN965_Pad, symbol Mechanical:MountingHole
- added H7, H8: MountingHole, MountingHole:MountingHole_5.3mm_M5_DIN965_Pad, symbol Mechanical:MountingHole

Commit message: Started work on new design with only one letter
Parts:
- removed C1: 0.1u, Capacitor_SMD:C_0603_1608Metric, symbol Device:C
- removed D30, D31, D32, D33, D34, D35, D36, D37, D38: LED, LED_THT:LED_D5.0mm, symbol Device:LED
- removed H7, H8: MountingHole, MountingHole:MountingHole_5.3mm_M5_DIN965_Pad, symbol Mechanical:MountingHole
- removed R30, R31, R32, R33, R34, R35, R36, R37, R38: 150, Resistor_SMD:R_0603_1608Metric, symbol Device:R
- removed U4: 74LS174, Package_DIP:DIP-16_W7.62mm, symbol 74xx:74LS174
- added H4: MountingHole, MountingHole:MountingHole_5.3mm_M5_DIN965_Pad, symbol Mechanical:MountingHole
Connections:
- net DATA is gone; now on net DATA_out_K: A1.5 (D2)
- no-connect marks 26 -> 25
Other:
- moved on the sheet: D39
