File: Ovve_Leds/A_letter.kicad_sch (KiCad schematic)
At the start: 46 parts, among them U1 74LS174

Commit message: Preliminarily finished with routing letter
Changed lines of the file:
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@@
 		)
 		(property "Value" "GND"
-			(at 50.8 76.2 0)
+			(at 48.26 72.39 0)
 			(effects
 				(font
